Commit message: copy values from 335Le URDF; change some frame names to be consistent with other cameras

File: orbbec_description/urdf/gemini335Le_macro.urdf.xacro (robot description, xacro)
@@ -1,5 +1,5 @@
 <?xml version="1.0" encoding="utf-8"?>
 <robot xmlns:xacro="http://ros.org/wiki/xacro">
-<!-- based off of https://github.com/orbbec/OrbbecSDK_ROS2/blob/v2-main/orbbec_description/urdf/gemini335L_336L.urdf.xarco -->
+<!-- based off of orbbec_description/urdf/gemini335Le.urdf.xacro -->
 <xacro:macro name="gemini_335L_336L" params="
     parent
@@ -20,9 +20,15 @@
     <inertial>
       <origin
-        xyz="0.00288 0.00062 0.01411"
+        xyz="0.01235 -0.0020872 0.013243"
         rpy="0 0 0" />
       <mass
-        value="0.03307" />
-      <inertia ixx="0.00004" ixy="0" ixz="0" iyy="0.000003" iyz="0" izz="0.00004" />
+        value="0.0.043446" />
+      <inertia
+        ixx="6.3353E-05"
+        ixy="-1.7904E-06"
+        ixz="-8.8334E-08"
+        iyy="8.2334E-06"
+        iyz="3.3581E-07"
+        izz="6.2898E-05" />
     </inertial>
     <visual>
@@ -32,11 +38,11 @@
       <geometry>
         <mesh
-          filename="file://$(find orbbec_description)/meshes/gemini335L_336L/base_link_simplified.stl" />
+          filename="file://$(find orbbec_description)/meshes/gemini335Le/base_link_simplified.stl" />
       </geometry>
-      <material
-        name="">
-        <color rgba="0.792 0.820 0.933 1" />
+      <material name="">
+        <color rgba="0.8 0.8 0.8 1" />
       </material>
     </visual>
+    <!-- TODO - set collision size -->
     <collision>
       <origin xyz="0 0 0.015" rpy="0 0 0" />
@@ -46,7 +52,7 @@
     </collision>
   </link>
-  <link name="${prefix}_color_screw_frame" />
+  <link name="${prefix}_bottom_screw_frame" />
   <joint
-    name="${prefix}_color_screw_frame_joint"
+    name="${prefix}_bottom_screw_frame_joint"
     type="fixed">
     <origin
@@ -56,33 +62,19 @@
       link="${prefix}_link" />
     <child
-      link="${prefix}_color_screw_frame" />
+      link="${prefix}_bottom_screw_frame" />
     <axis
       xyz="0 0 0" />
   </joint>
-  <link name="${prefix}_IMU_frame" />
+  <link name="${prefix}_infra2_frame" />
   <joint
-    name="${prefix}_IMU_frame_joint"
+    name="${prefix}_infra2_frame_joint"
     type="fixed">
     <origin
-      xyz="-0.002535 0.039634 0.013243"
+      xyz="0.034005 -0.0475 0.014048"
       rpy="0 0 0" />
     <parent
-      link="${prefix}_color_screw_frame" />
+      link="${prefix}_link" />
     <child
-      link="${prefix}_IMU_frame" />
-    <axis
-      xyz="0 0 0" />
-  </joint>
-  <link name="${prefix}_depth_frame" />
-  <joint
-    name="${prefix}_depth_frame_joint"
-    type="fixed">
-    <origin
-      xyz="0.011715 0.0475 0.014311"
-      rpy="0 0 0" />
-    <parent
-      link="${prefix}_color_screw_frame" />
-    <child
-      link="${prefix}_depth_frame" />
+      link="${prefix}_infra2_frame" />
     <axis
       xyz="0 0 0" />
@@ -93,8 +85,8 @@
     type="fixed">
     <origin
-      xyz="0.011715 0.0475 0.014311"
+      xyz="0.034005 0.0475 0.014048"
       rpy="0 0 0" />
     <parent
-      link="${prefix}_color_screw_frame" />
+      link="${prefix}_link" />
     <child
       link="${prefix}_infra1_frame" />
@@ -102,55 +94,13 @@
       xyz="0 0 0" />
   </joint>
-  <link name="${prefix}_infra1_optical_frame" />
+  <link name="${prefix}_color_frame" />
   <joint
-    name="${prefix}_infra1_optical_frame_joint"
+    name="${prefix}_frame_frame_joint"
     type="fixed">
     <origin
-      xyz="0 0 0"
-      rpy="-1.5708 0 -1.5708" />
-    <parent
-      link="${prefix}_infra1_frame" />
-    <child
-      link="${prefix}_infra1_optical_frame" />
-    <axis
-      xyz="0 0 0" />
-  </joint>
-  <link name="${prefix}_infra2_frame" />
-  <joint
-    name="${prefix}_infra2_frame_joint"
-    type="fixed">
-    <origin
-      xyz="0.011715 -0.0475 0.014311"
+      xyz="0.034014 0.02375 0.014048"
       rpy="0 0 0" />
     <parent
-      link="${prefix}_color_screw_frame" />
-    <child
-      link="${prefix}_infra2_frame" />
-    <axis
-      xyz="0 0 0" />
-  </joint>
-  <link name="${prefix}_infra2_optical_frame" />
-  <joint
-    name="${prefix}_infra2_optical_frame_joint"
-    type="fixed">
-    <origin
-      xyz="0 0 0"
-      rpy="-1.5708 0 -1.5708" />
-    <parent
-      link="${prefix}_infra2_frame" />
-    <child
-      link="${prefix}_infra2_optical_frame" />
-    <axis
-      xyz="0 0 0" />
-  </joint>
-  <link name="${prefix}_color_frame" />
-  <joint
-    name="${prefix}_color_frame_joint"
-    type="fixed">
-    <origin
-      xyz="0.011715 0.02375 0.014311"
-      rpy="0.0010157 0 0" />
-    <parent
-      link="${prefix}_color_screw_frame" />
+      link="${prefix}_link" />
     <child
       link="${prefix}_color_frame" />
@@ -158,15 +108,15 @@
       xyz="0 0 0" />
   </joint>
-  <link name="${prefix}_color_optical_frame" />
+  <link name="${prefix}_imu_frame" />
   <joint
-    name="${prefix}_color_optical_frame_joint"
+    name="${prefix}_imu_frame_joint"
     type="fixed">
     <origin
-      xyz="0 0 0"
-      rpy="-1.5708 0 -1.5708" />
+      xyz="0.019757 0.03619 0.013358"
+      rpy="0 0 0" />
     <parent
-      link="${prefix}_color_frame" />
+      link="${prefix}_link" />
     <child
-      link="${prefix}_color_optical_frame" />
+      link="${prefix}_imu_frame" />
     <axis
       xyz="0 0 0" />

Commit message: add optical frames

File: orbbec_description/urdf/gemini335Le_macro.urdf.xacro (robot description, xacro)
@@ -2,5 +2,5 @@
 <robot xmlns:xacro="http://ros.org/wiki/xacro">
 <!-- based off of orbbec_description/urdf/gemini335Le.urdf.xacro -->
-<xacro:macro name="gemini_335L_336L" params="
+<xacro:macro name="gemini_335Le" params="
     parent
     prefix:='camera'
@@ -44,5 +44,5 @@
       </material>
     </visual>
-    <!-- TODO - set collision size -->
+    <!-- TODO: set collision size -->
     <collision>
       <origin xyz="0 0 0.015" rpy="0 0 0" />
@@ -80,4 +80,18 @@
       xyz="0 0 0" />
   </joint>
+  <link name="${prefix}_infra2_optical_frame" />
+  <joint
+    name="${prefix}_infra2_optical_frame_joint"
+    type="fixed">
+    <origin
+      xyz="0 0 0"
+      rpy="-1.5708 0 -1.5708" />
+    <parent
+      link="${prefix}_infra2_frame" />
+    <child
+      link="${prefix}_infra2_optical_frame" />
+    <axis
+      xyz="0 0 0" />
+  </joint>
   <link name="${prefix}_infra1_frame" />
   <joint
@@ -91,4 +105,18 @@
     <child
       link="${prefix}_infra1_frame" />
+    <axis
+      xyz="0 0 0" />
+  </joint>
+  <link name="${prefix}_infra1_optical_frame" />
+  <joint
+    name="${prefix}_infra1_optical_frame_joint"
+    type="fixed">
+    <origin
+      xyz="0 0 0"
+      rpy="-1.5708 0 -1.5708" />
+    <parent
+      link="${prefix}_infra1_frame" />
+    <child
+      link="${prefix}_infra1_optical_frame" />
     <axis
       xyz="0 0 0" />
@@ -108,4 +136,18 @@
       xyz="0 0 0" />
   </joint>
+  <link name="${prefix}_color_optical_frame" />
+  <joint
+    name="${prefix}_color_optical_frame_joint"
+    type="fixed">
+    <origin
+      xyz="0 0 0"
+      rpy="-1.5708 0 -1.5708" />
+    <parent
+      link="${prefix}_color_frame" />
+    <child
+      link="${prefix}_color_optical_frame" />
+    <axis
+      xyz="0 0 0" />
+  </joint>
   <link name="${prefix}_imu_frame" />
   <joint
@@ -122,4 +164,5 @@
       xyz="0 0 0" />
   </joint>
+  <!-- TODO: check image properties for 335Le and 335L -->
   <xacro:if value="${sim_gazebo}">
     <!-- Use the realsense2_gz_description which can simulate a generic depth camera -->

Commit message: set collision size

File: orbbec_description/urdf/gemini335Le_macro.urdf.xacro (robot description, xacro)
@@ -23,5 +23,5 @@
         rpy="0 0 0" />
       <mass
-        value="0.0.043446" />
+        value="0.043446" />
       <inertia
         ixx="6.3353E-05"
@@ -44,9 +44,8 @@
       </material>
     </visual>
-    <!-- TODO: set collision size -->
     <collision>
-      <origin xyz="0 0 0.015" rpy="0 0 0" />
+      <origin xyz="0.013 0 0.015" rpy="0 0 0" />
       <geometry>
-        <box size="0.03 0.13 0.03"/>
+        <box size="0.055 0.125 0.03"/>
       </geometry>
     </collision>

Commit message: Add inertia and remove 'frame' from joint names

File: orbbec_description/urdf/gemini335Le_macro.urdf.xacro (robot description, xacro)
@@ -49,5 +49,5 @@
   <link name="${name}_bottom_screw_frame" />
   <joint
-    name="${name}_bottom_screw_frame_joint"
+    name="${name}_bottom_screw_joint"
     type="fixed">
     <origin
@@ -63,5 +63,5 @@
   <link name="${name}_infra2_frame" />
   <joint
-    name="${name}_infra2_frame_joint"
+    name="${name}_infra2_joint"
     type="fixed">
     <origin
@@ -77,5 +77,5 @@
   <link name="${name}_infra2_optical_frame" />
   <joint
-    name="${name}_infra2_optical_frame_joint"
+    name="${name}_infra2_optical_joint"
     type="fixed">
     <origin
@@ -91,5 +91,5 @@
   <link name="${name}_infra1_frame" />
   <joint
-    name="${name}_infra1_frame_joint"
+    name="${name}_infra1_joint"
     type="fixed">
     <origin
@@ -105,5 +105,5 @@
   <link name="${name}_infra1_optical_frame" />
   <joint
-    name="${name}_infra1_optical_frame_joint"
+    name="${name}_infra1_optical_joint"
     type="fixed">
     <origin
@@ -119,5 +119,5 @@
   <link name="${name}_depth_frame" />
   <joint
-    name="${name}_depth_frame_joint"
+    name="${name}_depth_joint"
     type="fixed">
     <parent
@@ -130,5 +130,5 @@
   <link name="${name}_depth_optical_frame" />
   <joint
-    name="${name}_depth_optical_frame_joint"
+    name="${name}_depth_optical_joint"
     type="fixed">
     <parent
@@ -139,7 +139,15 @@
       xyz="0 0 0" />
   </joint>
-  <link name="${name}_color_frame" />
+  <link name="${name}_color_frame" >
+    <inertial>
+        <mass value="0.01" />
+        <origin xyz="0 0 0" rpy="0 0 0"/>
+        <inertia ixx="0.001"  ixy="0" ixz="0"
+                 iyx="0" iyy="0.001" iyz="0"
+                 izx="0" izy="0" izz="0.001" />
+      </inertial>
+  </link>
   <joint
-    name="${name}_frame_frame_joint"
+    name="${name}_color_joint"
     type="fixed">
     <origin
@@ -155,5 +163,5 @@
   <link name="${name}_color_optical_frame" />
   <joint
-    name="${name}_color_optical_frame_joint"
+    name="${name}_color_optical_joint"
     type="fixed">
     <origin
@@ -169,5 +177,5 @@
   <link name="${name}_imu_frame" />
   <joint
-    name="${name}_imu_frame_joint"
+    name="${name}_imu_joint"
     type="fixed">
     <origin
