Commit message: add depth_frame and depth_optical_frame

File: orbbec_description/urdf/gemini335L_336L_macro.urdf.xacro (robot description, xacro)
@@ -88,4 +88,18 @@
       xyz="0 0 0" />
   </joint>
+  <link name="${prefix}_depth_optical_frame" />
+  <joint
+    name="${prefix}_depth_optical_frame_joint"
+    type="fixed">
+    <origin
+      xyz="0 0 0"
+      rpy="-1.5708 0 -1.5708" />
+    <parent
+      link="${prefix}_depth_frame" />
+    <child
+      link="${prefix}_depth_optical_frame" />
+    <axis
+      xyz="0 0 0" />
+  </joint>
   <link name="${prefix}_infra1_frame" />
   <joint

File: orbbec_description/urdf/gemini335Le_macro.urdf.xacro (robot description, xacro)
@@ -121,4 +121,26 @@
       xyz="0 0 0" />
   </joint>
+  <link name="${prefix}_depth_frame" />
+  <joint
+    name="${prefix}_depth_frame_joint"
+    type="fixed">
+    <parent
+      link="${prefix}_infra1_frame" />
+    <child
+      link="${prefix}_depth_frame" />
+    <axis
+      xyz="0 0 0" />
+  </joint>
+  <link name="${prefix}_depth_optical_frame" />
+  <joint
+    name="${prefix}_depth_optical_frame_joint"
+    type="fixed">
+    <parent
+      link="${prefix}_infra1_optical_frame" />
+    <child
+      link="${prefix}_depth_optical_frame" />
+    <axis
+      xyz="0 0 0" />
+  </joint>
   <link name="${prefix}_color_frame" />
   <joint

Commit message: frame_joint -> joint

File: orbbec_description/urdf/gemini335L_336L_macro.urdf.xacro (robot description, xacro)
@@ -44,5 +44,5 @@
   <link name="${prefix}_color_screw_frame" />
   <joint
-    name="${prefix}_color_screw_frame_joint"
+    name="${prefix}_color_screw_joint"
     type="fixed">
     <origin
@@ -58,5 +58,5 @@
   <link name="${prefix}_IMU_frame" />
   <joint
-    name="${prefix}_IMU_frame_joint"
+    name="${prefix}_IMU_joint"
     type="fixed">
     <origin
@@ -72,5 +72,5 @@
   <link name="${prefix}_depth_frame" />
   <joint
-    name="${prefix}_depth_frame_joint"
+    name="${prefix}_depth_joint"
     type="fixed">
     <origin
@@ -86,5 +86,5 @@
   <link name="${prefix}_depth_optical_frame" />
   <joint
-    name="${prefix}_depth_optical_frame_joint"
+    name="${prefix}_depth_optical_joint"
     type="fixed">
     <origin
@@ -100,5 +100,5 @@
   <link name="${prefix}_infra1_frame" />
   <joint
-    name="${prefix}_infra1_frame_joint"
+    name="${prefix}_infra1_joint"
     type="fixed">
     <origin
@@ -114,5 +114,5 @@
   <link name="${prefix}_infra1_optical_frame" />
   <joint
-    name="${prefix}_infra1_optical_frame_joint"
+    name="${prefix}_infra1_optical_joint"
     type="fixed">
     <origin
@@ -128,5 +128,5 @@
   <link name="${prefix}_infra2_frame" />
   <joint
-    name="${prefix}_infra2_frame_joint"
+    name="${prefix}_infra2_joint"
     type="fixed">
     <origin
@@ -142,5 +142,5 @@
   <link name="${prefix}_infra2_optical_frame" />
   <joint
-    name="${prefix}_infra2_optical_frame_joint"
+    name="${prefix}_infra2_optical_joint"
     type="fixed">
     <origin
@@ -156,5 +156,5 @@
   <link name="${prefix}_color_frame" />
   <joint
-    name="${prefix}_color_frame_joint"
+    name="${prefix}_color_joint"
     type="fixed">
     <origin
@@ -170,5 +170,5 @@
   <link name="${prefix}_color_optical_frame" />
   <joint
-    name="${prefix}_color_optical_frame_joint"
+    name="${prefix}_color_optical_joint"
     type="fixed">
     <origin

File: orbbec_description/urdf/gemini_335_336.urdf.xacro (robot description, xacro)
@@ -54,5 +54,5 @@
         </collision>
     </link>
-    <joint name="camera_bottom_screw_frame_joint" type="fixed">
+    <joint name="camera_bottom_screw_joint" type="fixed">
         <origin xyz="0 0 0" rpy="0 0 0" />
         <parent link="camera_link" />

Commit message: update 335L_336L with inertia

File: orbbec_description/urdf/gemini335L_336L_macro.urdf.xacro (robot description, xacro)
@@ -154,5 +154,13 @@
       xyz="0 0 0" />
   </joint>
-  <link name="${prefix}_color_frame" />
+  <link name="${prefix}_color_frame" >
+    <inertial>
+        <mass value="0.01" />
+        <origin xyz="0 0 0" rpy="0 0 0"/>
+        <inertia ixx="0.001"  ixy="0" ixz="0"
+                 iyx="0" iyy="0.001" iyz="0"
+                 izx="0" izy="0" izz="0.001" />
+      </inertial>
+  </link>
   <joint
     name="${prefix}_color_joint"
