Commit message: revert Orbbec defined urdf

File: orbbec_description/urdf/gemini_335_336.urdf.xacro (robot description, xacro)
@@ -54,5 +54,5 @@
         </collision>
     </link>
-    <joint name="camera_bottom_screw_joint" type="fixed">
+    <joint name="camera_bottom_screw_frame_joint" type="fixed">
         <origin xyz="0 0 0" rpy="0 0 0" />
         <parent link="camera_link" />
